File: pcb/bloop/bloop.kicad_pcb (KiCad board)
At the start: 2 copper layers, 0 parts

Commit message: Added BGT24MTR12 VQFN-32-9 footprint Updated gold material on 3d model 734153320
Other:
- net class 50ohm_24GHz added: clearance 0.5588, trace_width 0.540004, via_dia 0.8, via_drill 0.4
- rule trace_min: 0.2 -> 0.1016
- rule via_min_size: 0.4 -> 0.45
Changed lines of the file:
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@@
-(kicad_pcb (version 20171130) (host pcbnew "(5.1.2)-2")
+(kicad_pcb (version 20171130) (host pcbnew "(5.1.2)-1")
   (general
     (thickness 1.6)
@@
   (setup
     (last_trace_width 0.25)
+    (user_trace_width 0.540004)
     (trace_clearance 0.2)
     (zone_clearance 0.508)
     (zone_45_only no)
-    (trace_min 0.2)
+    (trace_min 0.1016)
     (via_size 0.8)
     (via_drill 0.4)
-    (via_min_size 0.4)
+    (via_min_size 0.45)
     (via_min_drill 0.3)
     (uvia_size 0.3)
@@
     (solder_mask_min_width 0.25)
     (aux_axis_origin 0 0)
-    (visible_elements FFFFEF7F)
+    (visible_elements 7FFFFFFF)
     (pcbplotparams
       (layerselection 0x010fc_ffffffff)
@@
     (via_dia 0.8)
     (via_drill 0.4)
+    (uvia_dia 0.3)
+    (uvia_drill 0.1)
+  )
+  (net_class 50ohm_24GHz ""
+    (clearance 0.5588)
+    (trace_width 0.540004)
+    (via_dia 0.8)
+    (via_drill 0.4)
