File: hardware/rf/rf/rf.sch (KiCad schematic (older format))
At the start: 27 parts

Commit message: Initial RF radar module schematic
Parts:
- removed FL?: LPF_35GHz, bloop:35GHz_LPF, symbol bloop:LPF_35GHz
- removed R?: R_US, symbol Device:R_US
- added C12, C21, C?: 10n, Capacitor_SMD:C_0402_1005Metric, symbol Device:C
- added C13: 2.2n, Capacitor_SMD:C_0402_1005Metric, symbol Device:C
- added C14, C19: 4.7u, Capacitor_SMD:C_0603_1608Metric, symbol Device:C
- added C16: ~, Capacitor_SMD:C_0402_1005Metric, symbol Device:C
- added C20: 1n, Capacitor_SMD:C_0402_1005Metric, symbol Device:C
- added C?: 100n, Capacitor_SMD:C_0402_1005Metric, symbol Device:C
- added FB1, FB2, FB3: Ferrite_Bead, Inductor_SMD:L_0402_1005Metric, symbol Device:Ferrite_Bead
- added FL1: LPF_35GHz, bloop:35GHz_LPF, symbol bloop:LPF_35GHz
- added J1: Conn_02x14_Odd_Even, symbol Connector_Generic:Conn_02x14_Odd_Even
- added J2, J3, J4: SMP, bloop:0734153320, symbol Connector:Conn_Coaxial
- added R1, R3, R9: 0, Resistor_SMD:R_0402_1005Metric, symbol Device:R_US
- added R10: 100, Resistor_SMD:R_0402_1005Metric, symbol Device:R_US
- added R8: 820, Resistor_SMD:R_0402_1005Metric, symbol Device:R_US
- C1, C10, C11, C2, C3, C4, C5, C6, C7, C8, C9: renamed from C?; footprint (none) -> Capacitor_SMD:C_0402_1005Metric
- C15: renamed from C?; value C -> 33n; footprint (none) -> Capacitor_SMD:C_0402_1005Metric
- C17, C18: renamed from C?; value 10n -> 1n; footprint (none) -> Capacitor_SMD:C_0402_1005Metric
- C22, C23: renamed from C?; footprint (none) -> bloop:DC_Block
- R2, R4, R5, R6: renamed from R?; footprint (none) -> Resistor_SMD:R_0402_1005Metric
- R7: renamed from R?; value R_US -> 120; footprint (none) -> Resistor_SMD:R_0402_1005Metric
- U1: renamed from U?; symbol rf-rescue:ECS-2520S-bloop -> bloop:ECS-2520S
- WLK1: renamed from WLK?; footprint (none) -> bloop:Wilk_AWR_Mod
- gave numbers to parts that had none: 2
Connections:
- net labels added: BGT24_ANA, GNDRF, IF1_I+, IF1_I-, IF1_Q+, IF1_Q-, IF2_I+, IF2_I-, IF2_Q+, IF2_Q-, PWR_IN, ~SPI_BGT24_CS, ~SPI_PLL_CS
- net labels removed: IF1_I, IF1_IX, IF1_Q, IF1_QX, IF2_I, IF2_IX, IF2_Q, IF2_QX, RX1, RX2, SPI_BGT24_CS, SPI_PLL_CS, TX
- wire segments 176 -> 271
- no-connect marks 1 -> 0
Other:
- note added: "CC"
- note added: "Castellated Pinout\n - VIN: +3.3 VDC (typ)\n - VIN: +3.6 VDC (max)\n - I = 265 mA (typ)\n - I = 325 mA (max)"
- note added: "I = 270 mA (max)"
- note added: "I = 55 mA (max)"
- note added: "I/Q"
- note added: "Oscillator"
- note added: "Power Flags"
- note added: "RF and Analog\nground isolated"
- note added: "RX1"
- note added: "RX2"
- note added: "TOTAL"
- note added: "TX"
- note added: "Zo"
- note removed: "Crystal oscillator"
- moved on the sheet: C1, C10, C11, C15, C17, C18, C2, C22, C23, C3, C4, C5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

Commit message: Corrected ~SPI_PLL_CS to PLL_LE and changed value of U1 to display the complete MPN
Parts:
- U1: value ECS-2520S -> ECS-2520S33-400
- gave numbers to parts that had none: 2
Connections:
- net labels added: PLL_LE
- net labels removed: ~SPI_PLL_CS
Changed lines of the file:
@@
 P 4400 7350
 F 0 "U1" H 4400 7750 50  0000 C CNN
-F 1 "ECS-2520S" H 4400 7000 50  0000 C CNN
+F 1 "ECS-2520S33-400" H 4400 7000 50  0000 C CNN
 F 2 "Crystal:Crystal_SMD_2520-4Pin_2.5x2.0mm" H 4400 7350 50  0001 C CNN
 F 3 "https://ecsxtal.com/store/pdf/ECS-2520S.pdf" H 4400 7350 50  0001 C CNN
@@
 SPI_MOSI
 Text Label 2750 5200 0    50   ~ 0
-~SPI_PLL_CS
+PLL_LE
 Text Label 2750 5400 0    50   ~ 0
 PLL_TRIG1
@@
 SPI_MOSI
 Text Label 6000 8300 0    50   ~ 0
-~SPI_PLL_CS
+PLL_LE
 Text Label 6000 8500 0    50   ~ 0
 PLL_TRIG1
@@
 	8750 1100 8750 1000
 $Comp
-L Device:C C?
+L Device:C C25
 U 1 1 5DA97864
 P 8750 1250
-F 0 "C?" H 8865 1296 50  0000 L CNN
+F 0 "C25" H 8865 1296 50  0000 L CNN
 F 1 "10n" H 8865 1205 50  0000 L CNN
 F 2 "Capacitor_SMD:C_0402_1005Metric" H 8788 1100 50  0001 C CNN
@@
 $EndComp
 $Comp
-L bloop:GNDRF #PWR?
+L bloop:GNDRF #PWR0101
 U 1 1 5DA9786A
 P 8750 1400
-F 0 "#PWR?" H 8750 1150 50  0001 C CNN
+F 0 "#PWR0101" H 8750 1150 50  0001 C CNN
 F 1 "GNDRF" H 8755 1227 50  0000 C CNN
 F 2 "" H 8750 1400 50  0001 C CNN
@@
 	8250 1100 8250 1000
 $Comp
-L Device:C C?
+L Device:C C24
 U 1 1 5DAAD4E3
 P 8250 1250
-F 0 "C?" H 8365 1296 50  0000 L CNN
+F 0 "C24" H 8365 1296 50  0000 L CNN
 F 1 "100n" H 8365 1205 50  0000 L CNN
 F 2 "Capacitor_SMD:C_0402_1005Metric" H 8288 1100 50  0001 C CNN
@@
 $EndComp
 $Comp
-L bloop:GNDRF #PWR?
+L bloop:GNDRF #PWR0102
 U 1 1 5DAAD4E9
 P 8250 1400
-F 0 "#PWR?" H 8250 1150 50  0001 C CNN
+F 0 "#PWR0102" H 8250 1150 50  0001 C CNN
 F 1 "GNDRF" H 8255 1227 50  0000 C CNN
 F 2 "" H 8250 1400 50  0001 C CNN
