File: hardware/rf/rf/rf.kicad_pcb (KiCad board)
At the start: 2 copper layers, 0 parts

Commit message: Setup board and layout parameters in pcbnew
Other:
- net class 50ohm_1.5GHz added: clearance 0.127, trace_width 0.5334, via_dia 0.8, via_drill 0.4
- net class 50ohm_24GHz added: clearance 0.127, trace_width 0.25, via_dia 0.8, via_drill 0.4
- net class Default: clearance 0.2 -> 0.1778; trace_width 0.25 -> 0.1778
- rule trace_clearance: 0.2 -> 0.1778
- rule trace_min: 0.2 -> 0.125
- rule via_min_drill: 0.3 -> 0.35
- rule via_min_size: 0.4 -> 0.6
Changed lines of the file:
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@@
 (kicad_pcb (version 20171130) (host pcbnew "(5.1.4)-1")
   (general
-    (thickness 1.6)
+    (thickness 0.32512)
     (drawings 0)
     (tracks 0)
@@
   (layers
     (0 F.Cu signal)
-    (31 B.Cu signal)
+    (31 B.Cu power)
     (32 B.Adhes user)
     (33 F.Adhes user)
@@
   )
   (setup
-    (last_trace_width 0.25)
-    (trace_clearance 0.2)
+    (last_trace_width 0.1778)
+    (trace_clearance 0.1778)
     (zone_clearance 0.508)
     (zone_45_only no)
-    (trace_min 0.2)
+    (trace_min 0.125)
     (via_size 0.8)
     (via_drill 0.4)
-    (via_min_size 0.4)
-    (via_min_drill 0.3)
+    (via_min_size 0.6)
+    (via_min_drill 0.35)
     (uvia_size 0.3)
     (uvia_drill 0.1)
@@
     (solder_mask_min_width 0.25)
     (aux_axis_origin 0 0)
-    (visible_elements FFFFFF7F)
+    (visible_elements 7FFFFFFF)
     (pcbplotparams
       (layerselection 0x010fc_ffffffff)
@@
   (net 0 "")
   (net_class Default "This is the default net class."
-    (clearance 0.2)
+    (clearance 0.1778)
+    (trace_width 0.1778)
+    (via_dia 0.8)
+    (via_drill 0.4)
+    (uvia_dia 0.3)
+    (uvia_drill 0.1)
+  )
+  (net_class 50ohm_1.5GHz ""
+    (clearance 0.127)
+    (trace_width 0.5334)
+    (via_dia 0.8)
+    (via_drill 0.4)
+    (uvia_dia 0.3)
+    (uvia_drill 0.1)
+  )
+  (net_class 50ohm_24GHz ""
+    (clearance 0.127)
     (trace_width 0.25)
     (via_dia 0.8)
