File: hardware/prototypes/spi_control/spi_control.sch (KiCad schematic (older format))
At the start: 0 parts

Commit message: Added MCP2210-L/MQ symbol and started schematic
Parts:
- added C? (x3): 100p, symbol Device:C
- added D? (x2): LED, symbol Device:LED
- added D?: SP0503BAHTG, digikey-footprints:SOT-143-4, symbol dk_TVS-Diodes:SP0503BAHTG
- added J?: USB_B_Micro, symbol Connector:USB_B_Micro
- added R?: 1M, symbol Device:R_US
- added R? (x2): 820, symbol Device:R_US
- added U?: MCP2210-I_MQ, Package_DFN_QFN:QFN-20-1EP_5x5mm_P0.65mm_EP3.35x3.35mm, symbol bloop:MCP2210-I_MQ
- added Y?: 12MHZ, symbol Device:Crystal
Connections:
- net labels added: GND, GNDPWR
- wire segments 0 -> 48
- no-connect marks 0 -> 1

Commit message: Added 3.3V LDO ST1L08SPU33R symbol. Completed power and SPI controller schematic sections
Parts:
- added C? (x3): 1u, symbol Device:C
- added C?: 4.7u, symbol Device:C
- added C?: 100n, symbol Device:C
- added D? (x2): GREEN_LED, symbol Device:LED
- added R? (x2): 330, symbol Device:R_US
- added R?: 1k, symbol Device:R_US
- added U?: ST1L08SPU33R, Package_DFN_QFN:DFN-8-1EP_2x3mm_P0.5mm_EP0.61x2.2mm, symbol bloop:ST1L08SPU33R
- C? (x2): value 100p -> 12p
- D? (x2): value LED -> GREEN_LED
- R?: value 820 -> 330
- Y?: footprint (none) -> Crystal:Crystal_SMD_Abracon_ABM8G-4Pin_3.2x2.5mm; MPN (none) -> ECS-120-12-33-AGN-TR
Connections:
- net labels added: +3.3V, 5V_USB, GNDREF, GPIO8, MISO, MOSI, PLL_CS, PLL_MOD, PLL_MUX, PLL_RSET, PLL_TRIG1, PLL_TRIG2, SCK, SPI_XFR, USB_D+, USB_D-, ~BGT_CS
- net labels removed: GNDPWR
- wire segments 48 -> 97
Other:
- note added: "12 mA (max)"
- note added: "3.3V GOOD"
- note added: "5V GOOD"
- note added: "Extra LED"
- note added: "SPI Controller"
- note added: "USB and +3.3V LDO"
- moved on the sheet: C?, D?, J?, R?, U?, Y?

Commit message: Added ADAR7251 symbol and ADC schematic sections
Parts:
- removed D?: GREEN_LED, symbol Device:LED
- removed R?: 330, symbol Device:R_US
- added C? (x14): C, symbol Device:C
- added C? (x2): 12p, symbol Device:C
- added C? (x2): 470n, symbol Device:C
- added C? (x9): 100n, symbol Device:C
- added C? (x8): 10u, symbol Device:C
- added C?: 1n, symbol Device:C
- added FB?: Ferrite_Bead, symbol Device:Ferrite_Bead
- added R?: R_US, symbol Device:R_US
- added R? (x3): 0, symbol Device:R_US
- added R? (x3): 10k, symbol Device:R_US
- added U? (x2): ADAR7251, Package_CSP:LFCSP-48-1EP_7x7mm_P0.5mm_EP4.1x4.1mm_ThermalVias, symbol bloop:ADAR7251
- added Y?: Crystal, symbol Device:Crystal
Connections:
- net labels added: +1V8, +3.3VA, ADC_DOUT0, ADC_DOUT1, ADC_DOUT2, ADC_DOUT3, ADC_DOUT4, ADC_DOUT5, ADC_DOUT6, ADC_DOUT7, BGT24_ANA, DATA_READY, GNDA, GNDD, IF1_I+, IF1_I-, IF1_Q+, IF1_Q-, IF2_I+, IF2_I-, IF2_Q+, IF2_Q-, MCLKIN, SCLK_ADC, ~ADC_CS, ~CONV_START, ~FAULT, ~RESET\PWDN
- net labels removed: GPIO8
- wire segments 97 -> 339
- no-connect marks 1 -> 2
Other:
- note added: "PLL Loop Filter"
- note added: "Power Flags"
- note removed: "Extra LED"
- moved on the sheet: C?, D?, J?, R?, U?, Y?

Commit message: Small schematic edits
Parts:
- added FB?: Ferrite_Bead, symbol Device:Ferrite_Bead
- added J?: Conn_01x25_Male, symbol Connector:Conn_01x25_Male
- C?: value 1u -> 4.7u
- C?: value C -> 5.6n
- C?: value C -> 390p
- R?: value R_US -> 1k
Connections:
- net labels removed: GNDD
- wire segments 339 -> 367
Other:
- note added: "TODO: Find a connector for these IO"
- moved on the sheet: D?
Changed lines of the file:
@@
 L power:GND #PWR?
 U 1 1 5DACD168
-P 5150 1750
-F 0 "#PWR?" H 5150 1500 50  0001 C CNN
-F 1 "GND" H 5155 1577 50  0000 C CNN
-F 2 "" H 5150 1750 50  0001 C CNN
-F 3 "" H 5150 1750 50  0001 C CNN
-	1    5150 1750
+P 5150 2100
+F 0 "#PWR?" H 5150 1850 50  0001 C CNN
+F 1 "GND" H 5155 1927 50  0000 C CNN
+F 2 "" H 5150 2100 50  0001 C CNN
+F 3 "" H 5150 2100 50  0001 C CNN
+	1    5150 2100
 	1    0    0    -1
 $EndComp
@@
 P 3250 1450
 F 0 "C?" H 3365 1496 50  0000 L CNN
-F 1 "1u" H 3365 1405 50  0000 L CNN
+F 1 "4.7u" H 3365 1405 50  0000 L CNN
 F 2 "" H 3288 1300 50  0001 C CNN
 F 3 "~" H 3250 1450 50  0001 C CNN
@@
 Connection ~ 5150 1700
 Wire Wire Line
-	5150 1700 5150 1750
+	5150 1700 5150 1950
 $Comp
 L Device:LED D?
 U 1 1 5DB2C8E5
-P 4700 2300
-F 0 "D?" V 4739 2182 50  0000 R CNN
-F 1 "GREEN_LED" V 4648 2182 50  0000 R CNN
-F 2 "" H 4700 2300 50  0001 C CNN
-F 3 "~" H 4700 2300 50  0001 C CNN
-	1    4700 2300
+P 4700 2500
+F 0 "D?" V 4739 2382 50  0000 R CNN
+F 1 "GREEN_LED" V 4648 2382 50  0000 R CNN
+F 2 "" H 4700 2500 50  0001 C CNN
+F 3 "~" H 4700 2500 50  0001 C CNN
+	1    4700 2500
 	0    -1   -1   0
 $EndComp
@@
 $EndComp
 Wire Wire Line
-	4700 2150 4700 2100
+	4700 2350 4700 2100
 Wire Wire Line
 	4550 1450 4700 1450
@@
 	4700 1450 4700 1800
 Wire Wire Line
-	4700 2450 4700 2500
+	4700 2650 4700 2700
 $Comp
 L power:GND #PWR?
 U 1 1 5DB4510F
-P 4700 2500
-F 0 "#PWR?" H 4700 2250 50  0001 C CNN
-F 1 "GND" H 4705 2327 50  0000 C CNN
-F 2 "" H 4700 2500 50  0001 C CNN
-F 3 "" H 4700 2500 50  0001 C CNN
-	1    4700 2500
-	1    0    0    -1
-$EndComp
-Text Notes 4850 2500 0    50   ~ 0
+P 4700 2700
+F 0 "#PWR?" H 4700 2450 50  0001 C CNN
+F 1 "GND" H 4705 2527 50  0000 C CNN
+F 2 "" H 4700 2700 50  0001 C CNN
+F 3 "" H 4700 2700 50  0001 C CNN
+	1    4700 2700
+	1    0    0    -1
+$EndComp
+Text Notes 4850 2700 0    50   ~ 0
 3.3V GOOD
 $Comp
@@
 Wire Notes Line
 	650  800  6500 800
-Text Notes 2350 750  0    100  ~ 20
+Text Notes 2800 750  0    100  ~ 20
 USB and +3.3V LDO
 $Comp
@@
 P 11550 7100
 F 0 "C?" H 11665 7146 50  0000 L CNN
-F 1 "C" H 11665 7055 50  0000 L CNN
+F 1 "5.6n" H 11665 7055 50  0000 L CNN
 F 2 "" H 11588 6950 50  0001 C CNN
 F 3 "~" H 11550 7100 50  0001 C CNN
@@
 P 12050 7300
 F 0 "C?" H 12165 7346 50  0000 L CNN
-F 1 "C" H 12165 7255 50  0000 L CNN
+F 1 "390p" H 12165 7255 50  0000 L CNN
 F 2 "" H 12088 7150 50  0001 C CNN
 F 3 "~" H 12050 7300 50  0001 C CNN
@@
 P 11550 7500
 F 0 "R?" H 11618 7546 50  0000 L CNN
-F 1 "R_US" H 11618 7455 50  0000 L CNN
+F 1 "1k" H 11618 7455 50  0000 L CNN
 F 2 "" V 11590 7490 50  0001 C CNN
 F 3 "~" H 11550 7500 50  0001 C CNN
@@
 	12700 3150 12700 3100
 Connection ~ 13050 3150
-$Comp
-L power:GNDD #PWR?
-U 1 1 5E058B2F
-P 12700 3200
-F 0 "#PWR?" H 12700 2950 50  0001 C CNN
-F 1 "GNDD" H 12704 3045 50  0000 C CNN
-F 2 "" H 12700 3200 50  0001 C CNN
-F 3 "" H 12700 3200 50  0001 C CNN
-	1    12700 3200
-	1    0    0    -1
-$EndComp
 Connection ~ 12700 3150
-$Comp
-L power:GNDD #PWR?
-U 1 1 5E05A0A5
-P 13050 2450
-F 0 "#PWR?" H 13050 2200 50  0001 C CNN
-F 1 "GNDD" H 13054 2295 50  0000 C CNN
-F 2 "" H 13050 2450 50  0001 C CNN
-F 3 "" H 13050 2450 50  0001 C CNN
-	1    13050 2450
-	1    0    0    -1
-$EndComp
 Wire Wire Line
 	12700 3200 12700 3150
@@
 $EndComp
 $Comp
-L power:PWR_FLAG #FLG?
-U 1 1 5F50D201
-P 3500 9950
-F 0 "#FLG?" H 3500 10025 50  0001 C CNN
-F 1 "PWR_FLAG" H 3500 10123 50  0000 C CNN
-F 2 "" H 3500 9950 50  0001 C CNN
-F 3 "~" H 3500 9950 50  0001 C CNN
-	1    3500 9950
-	1    0    0    -1
-$EndComp
-$Comp
 L power:GND #PWR?
 U 1 1 5F50D5E0
@@
 Wire Wire Line
 	3000 9950 3000 10150
-Wire Wire Line
-	3500 9950 3500 10150
-$Comp
-L power:GNDD #PWR?
-U 1 1 5F54A0C7
-P 3500 10150
-F 0 "#PWR?" H 3500 9900 50  0001 C CNN
-F 1 "GNDD" H 3504 9995 50  0000 C CNN
-F 2 "" H 3500 10150 50  0001 C CNN
-F 3 "" H 3500 10150 50  0001 C CNN
-	1    3500 10150
-	1    0    0    -1
-$EndComp
 $Comp
 L power:PWR_FLAG #FLG?
@@
 	2200 1250 2650 1250
 Wire Notes Line
-	700  9650 3800 9650
+	700  9650 3300 9650
 Wire Notes Line
-	3800 9650 3800 10450
+	3300 9650 3300 10450
 Wire Notes Line
-	3800 10450 700  10450
+	3300 10450 700  10450
 Wire Notes Line
 	700  10450 700  9650
@@
 Wire Wire Line
 	14200 2850 14250 2850
+$Comp
+L power:GND #PWR?
+U 1 1 5E8BDD0F
+P 13050 2450
+F 0 "#PWR?" H 13050 2200 50  0001 C CNN
+F 1 "GND" H 13055 2277 50  0000 C CNN
+F 2 "" H 13050 2450 50  0001 C CNN
+F 3 "" H 13050 2450 50  0001 C CNN
+	1    13050 2450
+	1    0    0    -1
+$EndComp
+$Comp
+L power:GND #PWR?
+U 1 1 5E8BE8CB
+P 12700 3200
+F 0 "#PWR?" H 12700 2950 50  0001 C CNN
+F 1 "GND" H 12705 3027 50  0000 C CNN
+F 2 "" H 12700 3200 50  0001 C CNN
+F 3 "" H 12700 3200 50  0001 C CNN
+	1    12700 3200
+	1    0    0    -1
+$EndComp
+$Comp
+L Device:Ferrite_Bead FB?
+U 1 1 5E8C0454
+P 5650 1950
+F 0 "FB?" V 5376 1950 50  0000 C CNN
+F 1 "Ferrite_Bead" V 5467 1950 50  0000 C CNN
+F 2 "" V 5580 1950 50  0001 C CNN
+F 3 "~" H 5650 1950 50  0001 C CNN
+	1    5650 1950
+	0    1    1    0
+$EndComp
+Wire Wire Line
+	5500 1950 5150 1950
+Connection ~ 5150 1950
+Wire Wire Line
+	5150 1950 5150 2100
+Wire Wire Line
+	5800 1950 6150 1950
+Wire Wire Line
+	6150 1950 6150 2100
+$Comp
+L power:GNDA #PWR?
+U 1 1 5E93EC78
+P 6150 2100
+F 0 "#PWR?" H 6150 1850 50  0001 C CNN
+F 1 "GNDA" H 6155 1927 50  0000 C CNN
+F 2 "" H 6150 2100 50  0001 C CNN
+F 3 "" H 6150 2100 50  0001 C CNN
+	1    6150 2100
+	1    0    0    -1
+$EndComp
+Wire Wire Line
+	14900 5400 14250 5400
+Wire Wire Line
+	14900 5300 14250 5300
+Wire Wire Line
+	14900 5200 14250 5200
+Wire Wire Line
+	14900 5100 14250 5100
+Wire Wire Line
+	14900 5000 14250 5000
+Text Label 14250 5800 0    50   ~ 0
+ADC_DOUT0
+Text Label 14250 5700 0    50   ~ 0
+ADC_DOUT1
+Text Label 14250 5600 0    50   ~ 0
+ADC_DOUT2
+Text Label 14250 5500 0    50   ~ 0
+ADC_DOUT3
+Text Label 14250 5400 0    50   ~ 0
+ADC_DOUT4
+Text Label 14250 5300 0    50   ~ 0
+ADC_DOUT5
+Text Label 14250 5200 0    50   ~ 0
+ADC_DOUT6
+Text Label 14250 5100 0    50   ~ 0
+ADC_DOUT7
+Text Label 14250 5000 0    50   ~ 0
+SCLK_ADC
+Wire Wire Line
+	14900 5800 14250 5800
+Wire Wire Line
+	14900 5700 14250 5700
+Wire Wire Line
+	14900 5600 14250 5600
+Wire Wire Line
+	14900 5500 14250 5500
+Wire Wire Line
+	14900 6300 14250 6300
+Wire Wire Line
+	14900 6000 14250 6000
+Wire Wire Line
+	14900 6100 14250 6100
+Text Label 14250 6300 0    50   ~ 0
+~CONV_START
+Text Label 14250 6200 0    50   ~ 0
+DATA_READY
+Text Label 14250 6100 0    50   ~ 0
+~FAULT
+Text Label 14250 6000 0    50   ~ 0
+~RESET\PWDN
+Wire Wire Line
+	14900 6200 14250 6200
+Wire Wire Line
+	14900 6700 14250 6700
+Text Label 14250 6800 0    50   ~ 0
+PLL_TRIG1
+Text Label 14250 6700 0    50   ~ 0
+PLL_TRIG2
+Wire Wire Line
+	14900 6600 14250 6600
+Text Label 14250 6600 0    50   ~ 0
+PLL_MOD
+Wire Wire Line
+	14900 6500 14250 6500
+Text Label 14250 6500 0    50   ~ 0
+PLL_MUX
+Wire Wire Line
+	14900 6400 14250 6400
+Text Label 14250 6400 0    50   ~ 0
+PLL_RSET
+Wire Wire Line
+	14900 6800 14250 6800
+Wire Wire Line
+	14900 7200 14250 7200
+Wire Wire Line
+	14900 7100 14250 7100
+Wire Wire Line
+	14900 7000 14250 7000
+Wire Wire Line
+	14900 6900 14250 6900
+Wire Wire Line
+	14900 7400 14250 7400
+Wire Wire Line
+	14900 7300 14250 7300
+Text Label 14250 6900 0    50   ~ 0
+MISO
+Text Label 14250 7000 0    50   ~ 0
+MOSI
+Text Label 14250 7100 0    50   ~ 0
+SCK
+Text Label 14250 7400 0    50   ~ 0
+PLL_CS
+Text Label 14250 7300 0    50   ~ 0
+~BGT_CS
+Text Label 14250 7200 0    50   ~ 0
+~ADC_CS
+Wire Wire Line
+	14900 5900 14250 5900
+Text Label 14250 5900 0    50   ~ 0
+MCLKIN
+$Comp
+L Connector:Conn_01x25_Male J?
+U 1 1 5EADE1E8
+P 15100 6200
+F 0 "J?" H 15072 6224 50  0000 R CNN
+F 1 "Conn_01x25_Male" H 15072 6133 50  0000 R CNN
+F 2 "" H 15100 6200 50  0001 C CNN
+F 3 "~" H 15100 6200 50  0001 C CNN
+	1    15100 6200
+	-1   0    0    -1
+$EndComp
+Text Notes 14000 4800 0    50   ~ 0
+TODO: Find a connector for these IO
 $EndSCHEMATC

Commit message: Copied the SP0503BA digikey symbol to project library and replaced in schematic
Parts:
- removed D?: SP0503BAHTG, digikey-footprints:SOT-143-4, symbol dk_TVS-Diodes:SP0503BAHTG
- added D?: SP0503BAHTG, Package_TO_SOT_SMD:SOT-143, symbol bloop:SP0503BAHTG
- U?: MPN (none) -> ST1L08SPU33R
Changed lines of the file:
@@
 NoConn ~ 1450 1650
-$Comp
-L dk_TVS-Diodes:SP0503BAHTG D?
-U 1 1 5DA2E4E9
-P 2250 2050
-F 0 "D?" H 2200 1703 60  0000 C CNN
-F 1 "SP0503BAHTG" H 2200 1809 60  0000 C CNN
-F 2 "digikey-footprints:SOT-143-4" H 2450 2250 60  0001 L CNN
-F 3 "https://www.littelfuse.com/~/media/files/littelfuse/technical%20resources/documents/data%20sheets/sp05xxba.pdf" H 2450 2350 60  0001 L CNN
-F 4 "F2715CT-ND" H 2450 2450 60  0001 L CNN "Digi-Key_PN"
-F 5 "SP0503BAHTG" H 2450 2550 60  0001 L CNN "MPN"
-F 6 "Circuit Protection" H 2450 2650 60  0001 L CNN "Category"
-F 7 "TVS - Diodes" H 2450 2750 60  0001 L CNN "Family"
-F 8 "https://www.littelfuse.com/~/media/files/littelfuse/technical%20resources/documents/data%20sheets/sp05xxba.pdf" H 2450 2850 60  0001 L CNN "DK_Datasheet_Link"
-F 9 "/product-detail/en/littelfuse-inc/SP0503BAHTG/F2715CT-ND/1154322" H 2450 2950 60  0001 L CNN "DK_Detail_Page"
-F 10 "TVS DIODE 5.5V 8.5V SOT143-4" H 2450 3050 60  0001 L CNN "Description"
-F 11 "Littelfuse Inc." H 2450 3150 60  0001 L CNN "Manufacturer"
-F 12 "Active" H 2450 3250 60  0001 L CNN "Status"
-	1    2250 2050
-	-1   0    0    1
-$EndComp
 $Comp
 L Device:C C?
@@
 F 2 "Package_DFN_QFN:DFN-8-1EP_2x3mm_P0.5mm_EP0.61x2.2mm" H 4200 1050 50  0001 C CNN
 F 3 "https://www.st.com/content/ccc/resource/technical/document/datasheet/5f/25/d1/3f/f8/25/44/07/DM00123507.pdf/files/DM00123507.pdf/jcr:content/translations/en.DM00123507.pdf" H 4150 1650 50  0001 C CNN
+F 4 "ST1L08SPU33R" H 4150 1450 50  0000 C CNN "MPN"
 	1    4150 1450
 	1    0    0    -1
@@
 Text Notes 14000 4800 0    50   ~ 0
 TODO: Find a connector for these IO
+$Comp
+L bloop:SP0503BAHTG D?
+U 1 1 5DB06C59
+P 2250 2050
+F 0 "D?" H 2200 1703 60  0000 C CNN
+F 1 "SP0503BAHTG" H 2200 1809 60  0000 C CNN
+F 2 "Package_TO_SOT_SMD:SOT-143" H 2450 2250 60  0001 L CNN
+F 3 "https://www.littelfuse.com/~/media/files/littelfuse/technical%20resources/documents/data%20sheets/sp05xxba.pdf" H 2450 2350 60  0001 L CNN
+F 4 "F2715CT-ND" H 2450 2450 60  0001 L CNN "Digi-Key_PN"
+F 5 "SP0503BAHTG" H 2450 2550 60  0001 L CNN "MPN"
+F 6 "Circuit Protection" H 2450 2650 60  0001 L CNN "Category"
+F 7 "TVS - Diodes" H 2450 2750 60  0001 L CNN "Family"
+F 8 "https://www.littelfuse.com/~/media/files/littelfuse/technical%20resources/documents/data%20sheets/sp05xxba.pdf" H 2450 2850 60  0001 L CNN "DK_Datasheet_Link"
+F 9 "/product-detail/en/littelfuse-inc/SP0503BAHTG/F2715CT-ND/1154322" H 2450 2950 60  0001 L CNN "DK_Detail_Page"
+F 10 "TVS DIODE 5.5V 8.5V SOT143-4" H 2450 3050 60  0001 L CNN "Description"
+F 11 "Littelfuse Inc." H 2450 3150 60  0001 L CNN "Manufacturer"
+F 12 "Active" H 2450 3250 60  0001 L CNN "Status"
+	1    2250 2050
+	-1   0    0    1
+$EndComp
 $EndSCHEMATC

Commit message: SPI schema 90%
Parts:
- added TP? (x6): TestPoint, TestPoint:TestPoint_Pad_D1.0mm, symbol Connector:TestPoint
- C1, C17, C18, C19, C2, C20, C21, C22, C23, C24, C27, C28, C29, C3, C30, C31, C32, C33, C34, C35, C36, C37, C38, C39, C4, C40, C41, C42, C43, C44: renamed from C?; footprint (none) -> Capacitor_SMD:C_0402_1005Metric
- C25, C26: renamed from C?; value 12p -> 18p; footprint (none) -> Capacitor_SMD:C_0402_1005Metric
- D2, D3, D4: renamed from D?; footprint (none) -> LED_SMD:LED_0402_1005Metric
- FB1, FB2: renamed from FB?; footprint (none) -> Inductor_SMD:L_0603_1608Metric
- R1, R10, R11, R12, R2, R3, R4, R5, R6, R7, R8, R9: renamed from R?; footprint (none) -> Resistor_SMD:R_0402_1005Metric
- Y2: renamed from Y?; value Crystal -> 40MHz; footprint (none) -> Oscillator:Oscillator_SMD_Abracon_ASE-4Pin_3.2x2.5mm; MPN (none) -> ECS-400-18-33-JGN-TR
- gave numbers to parts that had none: 19
Connections:
- net +3.3VA: now also TP?.1
- net +3V3: now also TP?.1, TP?.1
- net 5V_USB: now also TP?.1
- net GND: now also TP?.1
- net GNDA: now also TP?.1

Commit message: Include -rescue ignore from master anddelete -rescue byproducts; bring in BGT24 module symbols/footprints from master and add relevant 3D models; beautify spi_control.sch
Parts:
- removed TP? (x4): TestPoint, TestPoint:TestPoint_Pad_D1.0mm, symbol Connector:TestPoint
- added TP? (x5): TestPoint, TestPoint:TestPoint_Pad_D1.0mm, symbol Connector:TestPoint
- added U?: BGT24_Module, bloop:BGT24_Module, symbol bloop:BGT24_Module
- D3, D4: value GREEN_LED -> GRN
Connections:
- net +3.3VA: now also TP?.1
- net GND: now also TP?.1, TP?.1
- net GNDA: now also TP?.1
- net GNDREF: now also TP?.1
- new net: U?.1 (GND), U?.10 (GND), U?.13 (GND), U?.16 (GND), U?.17 (GND), U?.2 (GND), U?.20 (GND), U?.23 (GND), U?.29 (GND), U?.30 (GND), U?.7 (GND)
Other:
- note added: "4-Channel, 16-Bit, Continuous Time ADC"
- note added: "ADC Decoupling Bank"
- note added: "GND Test Points"
- note added: "Output Connector"
- note added: "SPI Transfer Activity"
- note added: "TODO: Find a connector\nfor these I/O"
- note removed: "TODO: Find a connector for these IO"
- moved on the sheet: C1, C10, C11, C12, C13, C14, C15, C16, C17, C18, C19, C2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

Commit message: Finished connector mapping for ECP5 devboard. Versa Connector.
Parts:
- removed J2: Conn_01x25_Male, symbol Connector:Conn_01x25_Male
- added J39: Versa_1, Connector_PinSocket_2.54mm:PinSocket_2x20_P2.54mm_Vertical_SMD, symbol Connector_Generic:Conn_02x20_Odd_Even
- added J40: Versa_2, Connector_PinSocket_2.54mm:PinSocket_2x20_P2.54mm_Vertical_SMD, symbol Connector_Generic:Conn_02x20_Odd_Even
- C10, C11, C12, C13, C14, C15, C16, C5, C6, C7, C8, C9: footprint (none) -> Capacitor_SMD:C_0402_1005Metric
- J1: footprint (none) -> Connector_USB:USB_Micro-B_Molex_47346-0001
- gave numbers to parts that had none: 8
Connections:
- net +3.3VA: now also U4.31 (PWR_IN), U4.32 (PWR_IN)
- net ADC_DOUT0: now also J39.18 (Pin_18)
- net ADC_DOUT1: now also J39.16 (Pin_16)
- net ADC_DOUT2: now also J39.14 (Pin_14)
- net ADC_DOUT3: now also J39.12 (Pin_12)
- net ADC_DOUT4: now also J39.10 (Pin_10)
- net ADC_DOUT5: now also J39.8 (Pin_8)
- net ADC_DOUT6: now also J39.6 (Pin_6)
- net ADC_DOUT7: now also J39.4 (Pin_4)
- net BGT24_ANA: now also U4.9 (BGT24_ANA)
- net DATA_READY: now also J40.1 (Pin_1)
- net GNDA: now also U4.1 (GND), U4.10 (GND), U4.13 (GND), U4.16 (GND), U4.17 (GND), U4.2 (GND), U4.20 (GND), U4.23 (GND), U4.29 (GND), U4.30 (GND), U4.7 (GND)
- net IF1_I+: now also U4.12 (IF1_I+)
- net IF1_I-: now also U4.11 (IF1_I-)
- net IF1_Q+: now also U4.14 (IF1_Q+)
- net IF1_Q-: now also U4.15 (IF1_Q-)
- net IF2_I+: now also U4.21 (IF2_I+)
- net IF2_I-: now also U4.22 (IF2_I-)
- net IF2_Q+: now also U4.19 (IF2_Q+)
- net IF2_Q-: now also U4.18 (IF2_Q-)
- net MCLKIN: now also J40.5 (Pin_5)
- net MISO: now also J39.11 (Pin_11)
- net MOSI: now also U4.5 (SPI_MOSI), J39.9 (Pin_9)
- net PLL_CS: now also U4.3 (SPI_CE_PLL), J39.17 (Pin_17)
- net PLL_MOD: now also U4.26 (PLL_MOD), J40.25 (Pin_25)
- net PLL_MUX: now also U4.25 (PLL_MUX), J40.23 (Pin_23)
- net PLL_RSET: now also J40.21 (Pin_21)
- net PLL_TRIG1: now also U4.28 (PLL_TRIG1), J40.29 (Pin_29)
- net PLL_TRIG2: now also U4.27 (PLL_TRIG2), J40.27 (Pin_27)
- net SCK: now also U4.4 (SPI_CLK), J39.7 (Pin_7)
- net SCLK_ADC: now also J39.5 (Pin_5)
- net ~ADC_CS: now also J40.31 (Pin_31)
- net ~BGT_CS: now also U4.24 (~SPI_BGT24_CS), J40.33 (Pin_33)
- net ~CONV_START: now also J39.29 (Pin_29)
- net ~FAULT: now also J39.31 (Pin_31)
- net ~RESET\PWDN: now also J39.33 (Pin_33)
- net F_IF2_Q+: now reaches C11.2, C15.2, U3.2 (AIN3P)
- net F_IF2_Q-: now reaches C15.1, C7.2, U3.3 (AIN3N)
- net F_IF2_I+: now reaches C12.2, C16.2, U3.4 (AIN4P)
- net F_IF1_Q+: now reaches C13.2, C9.2, U3.44 (AIN1P)
- net F_IF1_Q-: now reaches C13.1, C5.2, U3.45 (AIN1N)
- net F_IF1_I+: now reaches C10.2, C14.2, U3.46 (AIN2P)
- net F_IF1_I-: now reaches C14.1, C6.2, U3.47 (AIN2N)
- net F_IF2_I-: now reaches C16.1, C8.2, U3.5 (AIN4N)
- net PLL_LE: now reaches U4.6 (PLL_LE)
- net PLL_LE: now also J39.15 (Pin_15)
- net PLL_DIV_MCU: now reaches U4.8 (PLL_DIV_MCU)
- net PLL_DIV_MCU: now also J39.13 (Pin_13)
Other:
- note added: "Probably dont need these filters \nbased on ADAR72513 datasheet."
- note removed: "TODO: Find a connector\nfor these I/O"
- moved on the sheet: U4
